File: controller/splinktegrated.kicad_pcb (KiCad board)
At the start: 2 copper layers, 41.8 x 61.6 mm, 61 parts, among them J1 USB_C_Receptacle_USB2.0, J10 NA_Ribbon, J11 NA_Serial, J12 NA_Conn_01x04_Female, J14 Cirque, J2 NA_Conn_01x04_Female, J3 NA_Conn_01x04_Female, J4 NA_Conn_01x04_Female, J5 Conn_01x02, J6 Cirque, J7 NA_trackball, J8 NA_Ribbon, J9 NA_RGB, SW1 NA_SW_SPST, SW2 NA_SW_SPST, U1 RP2040, U2 USBLC6-2P6, U3 XC6210B332MR-G, U4 USBLC6-2P6, U5 W25Q128JVS, Y1 Crystal_GND24

Commit message: routing
Parts:
- removed J10: NA_Ribbon, Library:5_PinHeader
- removed J11: NA_Serial, drawings:Jack_3.5mm_PJ320E_Horizontal_custom
- removed J8: NA_Ribbon, Library:6_PinHeader
- removed NA_J6: Serial, drawings:Jack_3.5mm_PJ320E_Horizontal_custom
- removed NA_JP1, NA_JP2: NA_Jumper_2_Open, local-libraries:SolderJumper-2_P1.3mm_Open_RoundedPad1.0x1.5mm
- removed U2: USBLC6-2P6, Package_TO_SOT_SMD:SOT-666
Routing:
- net +3V3: track 134.7 -> 64.7 mm, vias 7 -> 3
- net col6_l: track 64.8 -> 0.00 mm, vias 3 -> 0
- net col5_l: track 62.4 -> 0.00 mm, vias 3 -> 0
- net col4_l: track 60.0 -> 0.00 mm, vias 3 -> 0
- net mosi_l: track 56.4 -> 0.00 mm, vias 2 -> 0
- net row5_l: track 56.3 -> 0.00 mm
- net row3_l: track 55.9 -> 0.00 mm, vias 3 -> 0
- net sc_l: track 53.8 -> 0.00 mm, vias 2 -> 0
- net row4_l: track 48.9 -> 0.00 mm, vias 2 -> 0
- net ss_l: track 47.1 -> 0.00 mm, vias 3 -> 0
- net miso_l: track 46.4 -> 0.00 mm, vias 2 -> 0
- net row2_l: track 46.1 -> 0.00 mm, vias 1 -> 0
- net col1_l: track 45.1 -> 0.00 mm, vias 1 -> 0
- net col2_l: track 40.7 -> 0.00 mm, vias 1 -> 0
- net row1_l: track 39.0 -> 0.00 mm, vias 1 -> 0
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
Commit message: work
Parts:
- removed J12, J4: NA_Conn_01x04_Female, drawings:PinHeader_1x04_P2.54mm_Vertical
- removed J14: Cirque, local-libraries:FPC-SMD_FPC05012-09200-.5mm
- removed J2, J3: NA_Conn_01x04_Female, Library:PinHeader_1x04_P2.54mm_Vertical_USB
- removed the J7 at (149.2, 113.6)
- removed J9: NA_RGB, Library:header1x03
- removed SW1: NA_SW_SPST, Library:PushSwitch
- added J11: Conn_01x07_Socket, Connector_PinSocket_2.54mm:PinSocket_1x07_P2.54mm_Vertical, F.Cu at (144.8, 111.8)
- H1, H2: footprint Library:MountingHole_4mm_Pad_Via -> drawings:MountingHole_3mm_Pad_Via
- SW2: moved to F.Cu
- moved H2 56.9 mm to (112.4, 100.6)
- moved J7 31.9 mm to (145.6, 100.4), turned to -90 degrees
- moved H1 28.7 mm to (118.2, 84.6)
- moved R9 11.9 mm to (146.0, 87.0), turned to 0 degrees
- moved C10 6.97 mm to (148.2, 87.0), turned to 0 degrees
- moved U5 4.75 mm to (148.7, 90.6), turned to 0 degrees
- moved R3 1.27 mm to (150.6, 103.2), turned to 90 degrees
- moved J5 0.81 mm to (150.2, 106.2)
- renumbered J6 to J7
Connections:
- net serial_l renamed /D1
- net split_hand_l renamed /D15
- J7 pad 1: +3V3 -> sc_l
- J7 pad 10: mosi_l -> SDA
- J7 pad 11: ss_l -> GND
- J7 pad 2: ss_l -> miso_l
- J7 pad 3: mosi_l -> NCS
- J7 pad 4: sc_l -> unconnected-(J7-Pin_4-Pad4)
- J7 pad 5: miso_l -> mosi_l
- J7 pad 6: GND -> unconnected-(J7-Pin_6-Pad6)
- J7 pad 7: GND -> unconnected-(J7-Pin_7-Pad7)
- J7 pad 8: miso_l -> unconnected-(J7-Pin_8-Pad8)
- J7 pad 9: sc_l -> SCL
- U1 pad 11: col6_l -> /D8
- U1 pad 12: row5_l -> /D9
- U1 pad 2: rgb_r -> /D0
- U1 pad 27: ss_l -> /D16
- U1 pad 32: col3_l -> NCS
- U1 pad 38: row2_l -> /A0
- U1 pad 39: col1_l -> /A1
- U1 pad 40: col2_l -> /A2
- U1 pad 41: row1_l -> /A3
- U1 pad 6: row4_l -> /D4
- U1 pad 7: row3_l -> /D5
- U1 pad 8: col4_l -> /D6
- U1 pad 9: col5_l -> /D7
Routing:
- net /~{RESET}: track 49.8 -> 25.8 mm, vias 2 -> 1
- net rgb_r: track 21.0 -> 0.00 mm
- net GND: track 43.5 -> 25.0 mm, vias 29 -> 26
- net +3V3: track 64.7 -> 46.2 mm
- net VBUS: track 29.1 -> 17.5 mm, vias 6 -> 4
- net /QSPI_~{CS}: track 19.4 -> 26.0 mm, vias 3 -> 2
- net /QSPI_D3: track 11.9 -> 5.54 mm
- net /QSPI_SCLK: track 9.97 -> 4.10 mm
- net /QSPI_D0: track 7.62 -> 2.67 mm
- net Net-(J1-SHIELD): track 14.4 -> 11.9 mm
- net /D-: track 15.5 -> 17.4 mm
- net /D+: track 15.9 -> 17.7 mm
- net /QSPI_D1: track 13.3 -> 11.7 mm
- net Net-(J1-CC1): track 3.16 -> 2.57 mm
- net /QSPI_D2: track 10.9 -> 10.4 mm
Other:
- board size 41.8 x 61.6 mm -> 20 x 41.6 mm

Commit message: work
Parts:
- SW2: moved to B.Cu
- moved G*** 60.5 mm to (197.6, 101.8)
- moved kibuzzard-61F01B61 60.5 mm to (201.1, 137.1)
- moved kibuzzard-6208EFFE 60.5 mm to (201.1, 137.5)
- moved G*** 50.8 mm to (171.3, 134.7)
- moved G*** 36.7 mm to (178.4, 120.8)
- moved G*** 26.9 mm to (176.9, 95.5)
- moved SW2 8.32 mm to (146.3, 99.5), turned to -90 degrees
- moved J11 1.20 mm to (144.8, 110.6)
Connections:
- J11 pad 1: unconnected-(J11-Pin_1-Pad1) -> sw1
- J11 pad 2: unconnected-(J11-Pin_2-Pad2) -> sw2
- J11 pad 3: unconnected-(J11-Pin_3-Pad3) -> sw3
- J11 pad 4: unconnected-(J11-Pin_4-Pad4) -> sw4
- J7 pad 10: SDA -> unconnected-(J7-Pin_10-Pad10)
- J7 pad 9: SCL -> unconnected-(J7-Pin_9-Pad9)
- U1 pad 11: /D8 -> sw3
- U1 pad 12: /D9 -> sw4
- U1 pad 18: /D15 -> unconnected-(U1-GPIO15-Pad18)
- U1 pad 2: /D0 -> unconnected-(U1-GPIO0-Pad2)
- U1 pad 27: /D16 -> unconnected-(U1-GPIO16-Pad27)
- U1 pad 3: /D1 -> unconnected-(U1-GPIO1-Pad3)
- U1 pad 38: /A0 -> unconnected-(U1-GPIO26_ADC0-Pad38)
- U1 pad 39: /A1 -> unconnected-(U1-GPIO27_ADC1-Pad39)
- U1 pad 40: /A2 -> unconnected-(U1-GPIO28_ADC2-Pad40)
- U1 pad 41: /A3 -> unconnected-(U1-GPIO29_ADC3-Pad41)
- U1 pad 6: /D4 -> unconnected-(U1-GPIO4-Pad6)
- U1 pad 7: /D5 -> unconnected-(U1-GPIO5-Pad7)
- U1 pad 8: /D6 -> sw1
- U1 pad 9: /D7 -> sw2
Routing:
- net NCS: track 0.00 -> 38.0 mm, vias 0 -> 2
- net sc_l: track 0.00 -> 37.7 mm
- net mosi_l: track 0.00 -> 36.8 mm
- net miso_l: track 0.00 -> 36.5 mm
- net +3V3: track 46.2 -> 71.1 mm, vias 3 -> 4
- net sw1: track 0.00 -> 24.5 mm, vias 0 -> 2
- net sw2: track 0.00 -> 23.5 mm, vias 0 -> 2
- net GND: track 25.0 -> 45.1 mm, vias 26 -> 28
- net /~{RESET}: track 25.8 -> 29.3 mm
- net /QSPI_D1: track 11.7 -> 14.4 mm
- net /QSPI_D2: track 10.4 -> 12.9 mm
- net /QSPI_~{CS}: track 26.0 -> 28.5 mm
- net /LED: track 12.4 -> 11.3 mm

Commit message: work
Parts:
- moved J11 2.02 mm to (144.8, 112.6)
- moved R3 0.51 mm to (150.1, 103.3)
- moved J5 0.40 mm to (149.8, 106.2)
- moved C1 0.37 mm to (161.2, 88.0)
- moved C9 0.10 mm to (149.2, 100.5)
Connections:
- J11 pad 5: unconnected-(J11-Pin_5-Pad5) -> GND
- J11 pad 6: unconnected-(J11-Pin_6-Pad6) -> RGB
- J11 pad 7: unconnected-(J11-Pin_7-Pad7) -> +3V3
- U1 pad 13: unconnected-(U1-GPIO10-Pad13) -> RGB
Routing:
- net GND: track 45.1 -> 129.2 mm, vias 28 -> 31
- net RGB: track 0.00 -> 16.9 mm, vias 0 -> 1
- net sw3: track 0.00 -> 16.3 mm, vias 0 -> 1
- net sw4: track 0.00 -> 14.5 mm, vias 0 -> 1
- net +3V3: track 71.1 -> 80.6 mm, vias 4 -> 5
- net miso_l: track 36.5 -> 39.8 mm
- net NCS: track 38.0 -> 41.4 mm
- net mosi_l: track 36.8 -> 40.1 mm
- net sc_l: track 37.7 -> 41.1 mm
- net /~{RESET}: track 29.3 -> 32.3 mm
- net sw2: track 23.5 -> 25.3 mm
- net sw1: track 24.5 -> 26.2 mm
- net +5V: track 6.88 -> 7.76 mm
- net /QSPI_~{CS}: track 28.5 -> 29.1 mm
- net /D+: track 17.7 -> 18.4 mm
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
Commit message: work
Parts:
- moved G*** 42.6 mm to (147.3, 99.5), turned to 180 degrees
- moved G*** 34.9 mm to (146.1, 107.6)
- moved G*** 29.4 mm to (148.3, 88.9)
Other:
- board text added: "3v3"
- board text added: "ARGOS CONTROLLER REV 1.0"
- board text added: "DESIGN BY Q. LEBASTARD BASTARDKB 2024"
- board text added: "SW1"
- board text added: "SW2"
- board text added: "SW3"
- board text added: "SW4"
- board text removed: "Compatible with splinky v3"
- board text removed: "DESIGN BY QUENTIN LEBASTARD BASTARDKB 2023"
- board text removed: "SPLINKTEGRATED REV 1.4"

Commit message: work
Parts:
- removed the G*** at (146.1, 107.6)
- J11: footprint Connector_PinSocket_2.54mm:PinSocket_1x07_P2.54mm_Vertical -> Library:PinSocket_1x07_P2.54mm_Vertical
Other:
- board size 20 x 41.6 mm -> 23 x 38.2 mm

Commit message: work
Other:
- board size 23 x 38.2 mm -> 23 x 41.6 mm
Changed lines of the file:
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@@
 	(gr_line
 		(start 162.3699 77.47)
-		(end 162.375 113.125)
+		(end 162.371945 116.501945)
+		(stroke
+			(width 0.1)
+			(type default)
+		)
+		(layer "Edge.Cuts")
+	)
+	(gr_arc
+		(start 150.91 117.775)
+		(mid 152.41 116.275)
+		(end 153.91 117.775)
 		(stroke
 			(width 0.1)
@@
 	(gr_line
 		(start 142.3949 109.065)
-		(end 142.4 113.13)
+		(end 142.4 116.501945)
 		(stroke
 			(width 0.1)
@@
 	)
 	(gr_line
+		(start 143.67 117.771945)
+		(end 150.91 117.775)
+		(stroke
+			(width 0.1)
+			(type default)
+		)
+		(layer "Edge.Cuts")
+	)
+	(gr_line
 		(start 147.79 76.205)
 		(end 143.6649 76.2)
@@
 		(layer "Edge.Cuts")
 	)
-	(gr_line
-		(start 143.67 114.4)
-		(end 161.105 114.395)
-		(stroke
-			(width 0.1)
-			(type default)
-		)
-		(layer "Edge.Cuts")
-	)
 	(gr_arc
-		(start 162.375 113.125)
-		(mid 162.003055 114.023055)
-		(end 161.105 114.395)
+		(start 162.371945 116.501945)
+		(mid 162 117.4)
+		(end 161.101945 117.771945)
 		(stroke
 			(width 0.1)
@@
 	)
 	(gr_line
+		(start 153.91 117.775)
+		(end 161.101945 117.771945)
+		(stroke
+			(width 0.1)
+			(type default)
+		)
+		(layer "Edge.Cuts")
+	)
+	(gr_line
 		(start 139.4 93.7)
 		(end 139.4 106.525)
@@
 	)
 	(gr_arc
-		(start 143.67 114.4)
-		(mid 142.771945 114.028055)
-		(end 142.4 113.13)
+		(start 143.67 117.771945)
+		(mid 142.771945 117.4)
+		(end 142.4 116.501945)
 		(stroke
 			(width 0.1)
@@
 		(layer "Edge.Cuts")
 	)
+	(gr_circle
+		(center 152.41 117.775)
+		(end 155.4 117.2)
+		(stroke
+			(width 0.15)
+			(type default)
+		)
+		(fill none)
+		(layer "Margin")
+	)
 	(gr_text "C3"

Commit message: VIK
Parts:
- removed the G*** at (197.6, 101.8)
- removed kibuzzard-61F01B61: G***, kibuzzard-61F01B61
- removed kibuzzard-6208EFFE: G***, kibuzzard-6208EFFE
- added J2: Conn_01x04_Socket, Connector_PinSocket_2.54mm:PinSocket_1x04_P2.54mm_Vertical, F.Cu at (163.2, 97.6)
- added JP1: Jumper_2_Bridged, Jumper:SolderJumper-2_P1.3mm_Open_RoundedPad1.0x1.5mm, F.Cu at (128.3, 77.8)
- moved H2 10.1 mm to (120.1, 94.1)
- moved H1 3.19 mm to (120.1, 82.0)
Connections:
- J7 pad 1: sc_l -> /SCLK
- J7 pad 10: unconnected-(J7-Pin_10-Pad10) -> SDA
- J7 pad 2: miso_l -> /MISO
- J7 pad 4: unconnected-(J7-Pin_4-Pad4) -> /A1
- J7 pad 5: mosi_l -> /MOSI
- J7 pad 6: unconnected-(J7-Pin_6-Pad6) -> /A0
- J7 pad 7: unconnected-(J7-Pin_7-Pad7) -> Net-(J7-Pin_7)
- J7 pad 8: unconnected-(J7-Pin_8-Pad8) -> RGB
- J7 pad 9: unconnected-(J7-Pin_9-Pad9) -> SCL
- U1 pad 13: RGB -> SDA
- U1 pad 14: unconnected-(U1-GPIO11-Pad14) -> SCL
- U1 pad 15: unconnected-(U1-GPIO12-Pad15) -> /MISO
- U1 pad 16: unconnected-(U1-GPIO13-Pad16) -> NCS
- U1 pad 17: unconnected-(U1-GPIO14-Pad17) -> /SCLK
- U1 pad 18: unconnected-(U1-GPIO15-Pad18) -> /MOSI
- U1 pad 31: miso_l -> unconnected-(U1-GPIO20-Pad31)
- U1 pad 32: NCS -> unconnected-(U1-GPIO21-Pad32)
- U1 pad 34: sc_l -> /SCLK
- U1 pad 35: mosi_l -> unconnected-(U1-GPIO23-Pad35)
- U1 pad 37: unconnected-(U1-GPIO25-Pad37) -> RGB
- U1 pad 38: unconnected-(U1-GPIO26_ADC0-Pad38) -> /A0
- U1 pad 39: unconnected-(U1-GPIO27_ADC1-Pad39) -> /A1
Routing:
- net NCS: track 41.4 -> 0.00 mm, vias 2 -> 0
- net sc_l: track 41.1 -> 0.00 mm
- net mosi_l: track 40.1 -> 0.00 mm
- net miso_l: track 39.8 -> 0.00 mm
Other:
- board size 23 x 41.6 mm -> 26 x 41.6 mm
- board text removed: "3.3V"
- board text removed: "C1"
- board text removed: "C2"
- board text removed: "C3"
- board text removed: "C4"
- board text removed: "C5"
- board text removed: "C6"
- board text removed: "MATRIX"
- board text removed: "MI"
- board text removed: "MO"
- board text removed: "R1"
- board text removed: "R2"
- board text removed: "R3"
- board text removed: "R4"
- board text removed: "R5"
- board text removed: "REV1.4"
- board text removed: "SC"
- board text removed: "SS"
- board text removed: "TRCK"
- board text removed: "USB board on THIS side for Left"
- board text removed: "USB board on THIS side for Right"
- board text removed: "this side not visible"
