File: controller/splinktegrated.kicad_pcb (KiCad board)
At the start: 2 copper layers, 26 x 41.6 mm, 45 parts, among them J1 USB_C_Receptacle_USB2.0, J11 Conn_01x07_Socket, J2 Conn_01x04_Socket, J5 Conn_01x02, J7 Cirque, SW2 NA_SW_SPST, U1 RP2040, U3 XC6210B332MR-G, U4 USBLC6-2P6, U5 W25Q128JVS, Y1 Crystal_GND24

Commit message: work
Parts:
- moved JP1 35.6 mm to (146.1, 108.5), turned to 90 degrees
Changed lines of the file:
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@@
 	(footprint "Jumper:SolderJumper-2_P1.3mm_Open_RoundedPad1.0x1.5mm"
 		(layer "F.Cu")
-		(at 128.268109 77.768109)
+		(at 146.1 108.55 90)
 		(descr "SMD Solder Jumper, 1x1.5mm, rounded Pads, 0.3mm gap, open")
 		(tags "solder jumper open")
 		(property "Reference" "JP1"
-			(at 0 -1.8 0)
+			(at 0 -1.8 270)
 			(layer "F.SilkS")
 			(effects
@@
 		)
 		(property "Value" "Jumper_2_Bridged"
-			(at 0 1.9 0)
+			(at 0 1.9 270)
 			(layer "F.Fab")
 			(effects
@@
 		)
 		(property "Footprint" "Jumper:SolderJumper-2_P1.3mm_Open_RoundedPad1.0x1.5mm"
-			(at 0 0 0)
+			(at 0 0 90)
 			(unlocked yes)
 			(layer "F.Fab")
@@
 		)
 		(property "Datasheet" ""
-			(at 0 0 0)
+			(at 0 0 90)
 			(unlocked yes)
 			(layer "F.Fab")
@@
 		)
 		(property "Description" ""
-			(at 0 0 0)
+			(at 0 0 90)
 			(unlocked yes)
 			(layer "F.Fab")
@@
 		(attr exclude_from_pos_files)
 		(fp_line
+			(start -0.7 -1)
+			(end 0.7 -1)
+			(stroke
+				(width 0.12)
+				(type solid)
+			)
+			(layer "F.SilkS")
+		)
+		(fp_line
+			(start 1.4 -0.3)
+			(end 1.4 0.3)
+			(stroke
+				(width 0.12)
+				(type solid)
+			)
+			(layer "F.SilkS")
+		)
+		(fp_line
 			(start -1.4 0.3)
 			(end -1.4 -0.3)
@@
 		)
 		(fp_line
-			(start -0.7 -1)
-			(end 0.7 -1)
-			(stroke
-				(width 0.12)
-				(type solid)
-			)
-			(layer "F.SilkS")
-		)
-		(fp_line
 			(start 0.7 1)
 			(end -0.7 1)
@@
 			(layer "F.SilkS")
 		)
-		(fp_line
-			(start 1.4 -0.3)
-			(end 1.4 0.3)
+		(fp_arc
+			(start 0.7 -1)
+			(mid 1.194975 -0.794975)
+			(end 1.4 -0.3)
 			(stroke
 				(width 0.12)
@@
 		)
 		(fp_arc
+			(start 1.4 0.3)
+			(mid 1.194975 0.794975)
+			(end 0.7 1)
+			(stroke
+				(width 0.12)
+				(type solid)
+			)
+			(layer "F.SilkS")
+		)
+		(fp_arc
 			(start -0.7 1)
 			(mid -1.194975 0.794975)
@@
 			(layer "F.SilkS")
 		)
-		(fp_arc
-			(start 0.7 -1)
-			(mid 1.194975 -0.794975)
-			(end 1.4 -0.3)
-			(stroke
-				(width 0.12)
-				(type solid)
-			)
-			(layer "F.SilkS")
-		)
-		(fp_arc
-			(start 1.4 0.3)
-			(mid 1.194975 0.794975)
-			(end 0.7 1)
-			(stroke
-				(width 0.12)
-				(type solid)
-			)
-			(layer "F.SilkS")
+		(fp_line
+			(start -1.65 -1.25)
+			(end 1.65 -1.25)
+			(stroke
+				(width 0.05)
+				(type solid)
+			)
+			(layer "F.CrtYd")
 		)
 		(fp_line
@@
 		)
 		(fp_line
-			(start -1.65 -1.25)
+			(start 1.65 1.25)
 			(end 1.65 -1.25)
 			(stroke
@@
 			(layer "F.CrtYd")
 		)
-		(fp_line
-			(start 1.65 1.25)
-			(end 1.65 -1.25)
-			(stroke
-				(width 0.05)
-				(type solid)
-			)
-			(layer "F.CrtYd")
-		)
 		(pad "1" smd custom
-			(at -0.65 0)
+			(at -0.65 0 90)
 			(size 1 0.5)
 			(layers "F.Cu" "F.Mask")
@@
 		)
 		(pad "2" smd custom
-			(at 0.65 0)
+			(at 0.65 0 90)
 			(size 1 0.5)
 			(layers "F.Cu" "F.Mask")

Commit message: work
Parts:
- removed R10: 5.1k, Resistor_SMD:R_0402_1005Metric
- removed R11: 10k, Resistor_SMD:R_0402_1005Metric
Connections:
- net /A0 renamed /GP26
- net /A1 renamed /GP27
- U1 pad 30: /VBUS_DET -> unconnected-(U1-GPIO19-Pad30)
Routing:
- net /VBUS_DET: track 15.1 -> 0.00 mm, vias 2 -> 0
- net VBUS: track 17.0 -> 9.98 mm
- net GND: track 129.2 -> 128.5 mm

Commit message: work
Parts:
- moved JP1 16.3 mm to (141.7, 92.8), turned to -90 degrees
- moved J2 7.97 mm to (163.3, 105.5), turned to 180 degrees
- moved J5 0.80 mm to (149.0, 106.2)
- moved R3 0.66 mm to (149.4, 103.2)
- moved C14 0.49 mm to (156.9, 104.2)
- moved C8 0.49 mm to (156.9, 103.1)
- moved D1 0.49 mm to (156.9, 106.4)
- moved R1 0.49 mm to (156.9, 105.3)
Connections:
- U1 pad 17: /SCLK -> unconnected-(U1-GPIO14-Pad17)
Routing:
- net /GP27: track 0.00 -> 59.2 mm
- net /SCLK: track 0.00 -> 54.6 mm, vias 0 -> 2
- net /GP26: track 0.00 -> 42.7 mm, vias 0 -> 2
- net SCL: track 0.00 -> 42.7 mm, vias 0 -> 1
- net SDA: track 0.00 -> 42.2 mm, vias 0 -> 1
- net +3V3: track 80.6 -> 119.8 mm, vias 5 -> 10
- net NCS: track 0.00 -> 36.8 mm, vias 0 -> 2
- net RGB: track 16.9 -> 49.4 mm, vias 1 -> 0
- net /MISO: track 0.00 -> 21.7 mm, vias 0 -> 2
- net /MOSI: track 0.00 -> 21.4 mm, vias 0 -> 2
- net /~{RESET}: track 32.3 -> 48.2 mm
- net Net-(J7-Pin_7): track 0.00 -> 12.0 mm, vias 0 -> 2
- net sw2: track 25.3 -> 33.3 mm, vias 2 -> 1
- net sw1: track 26.2 -> 32.8 mm, vias 2 -> 1
- net sw4: track 14.5 -> 15.4 mm
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Other:
- outline, holes or cut-outs redrawn

Commit message: work
Parts:
- moved G*** 1.53 mm to (146.8, 89.2)
Routing:
- net /GP27: track 59.2 -> 54.9 mm, vias 0 -> 2
- net /~{RESET}: track 48.2 -> 45.8 mm
- net sw1: track 32.8 -> 30.9 mm
- net sw2: track 33.3 -> 31.5 mm
- net /SCLK: track 54.6 -> 53.3 mm
- net /MISO: track 21.7 -> 20.4 mm
- net RGB: track 49.4 -> 48.1 mm
- net /MOSI: track 21.4 -> 22.4 mm
- net NCS: track 36.8 -> 35.9 mm
- net /LED: track 11.5 -> 12.1 mm
Other:
- board text added: "IO26"
- board text added: "IO27"
- board text added: "SCL"
- board text added: "SDA"

Commit message: work
Parts:
- removed the G*** at (147.3, 99.5)
- removed SW2: NA_SW_SPST, Library:PushSwitch
- added G***: LOGO, LOGO, F.Cu at (149.0, 105.7)
- added G***: LOGO, LOGO, F.Cu at (163.3, 101.8)
- added G***: LOGO, LOGO, F.Cu at (152.4, 112.6)
- added G***: LOGO, LOGO, B.Cu at (152.4, 112.6)
- added G***: LOGO, LOGO, B.Cu at (149.0, 105.7)
- added G***: LOGO, LOGO, B.Cu at (163.3, 101.8)
- J2: footprint Connector_PinSocket_2.54mm:PinSocket_1x04_P2.54mm_Vertical -> Library:PinSocket_1x04_P2.54mm_Vertical
- moved G*** 5.73 mm to (152.4, 90.2)
Routing:
- net /~{RESET}: track 45.8 -> 0.00 mm, vias 1 -> 0

Commit message: work
Connections:
- net VBUS renamed /Vbus_daughter
Routing:
- net /~{RESET}: track 0.00 -> 3.55 mm

Commit message: work
Other:
- board text added: "github.com/bastardkb"

Commit message: details
Parts:
- removed H1, H2: NA_M4, drawings:MountingHole_3mm_Pad_Via
