File: flex/flex.kicad_pcb (KiCad board)
At the start: 2 copper layers, 127 x 94.5 mm, 11 parts, among them J7 Conn_01x07_Socket, SW5 SW_Push, SW6 SW_Push, SW7 SW_Push, SW8 SW_Push

Commit message: flex PCB
Parts:
- moved J7 115.1 mm to (-97.3, 130.7), turned to 90 degrees
- moved C3 114.6 mm to (-78.8, 134.7), turned to 90 degrees
- moved R3 101.6 mm to (-76.6, 134.7)
- moved SW7 58.6 mm to (-68.9, 125.0)
- moved D16 58.6 mm to (-68.9, 129.6)
- moved SW6 53.6 mm to (-92.2, 119.4)
- moved D13 53.6 mm to (-92.2, 124.0)
- moved SW5 44.5 mm to (-92.2, 100.5)
- moved D14 44.5 mm to (-92.2, 105.1)
- moved SW8 38.5 mm to (-68.9, 106.2)
- moved D15 38.5 mm to (-68.9, 110.8)
- renumbered D14 to D13, D13 to D14
Connections:
- D13 pad 1: Net-(D14-DOUT) -> Net-(D13-DOUT)
- D13 pad 3: Net-(D13-DOUT) -> Net-(D13-DIN)
- D14 pad 1: Net-(D13-DOUT) -> Net-(D14-DOUT)
- D14 pad 3: Net-(D13-DIN) -> Net-(D13-DOUT)
- SW5 pad 1: sw1 -> sw2
- SW6 pad 1: sw3 -> sw1
- SW7 pad 1: sw2 -> sw4
- SW8 pad 1: sw4 -> sw3
Routing:
- net Gnd: track 0.00 -> 189.1 mm, vias 0 -> 7
- net Vcc: track 0.00 -> 149.4 mm
- net Net-(D14-DOUT): track 0.00 -> 128.4 mm, vias 0 -> 2
- net Net-(D15-DOUT): track 0.00 -> 73.1 mm, vias 0 -> 2
- net Net-(D13-DOUT): track 0.00 -> 66.3 mm, vias 0 -> 2
- net sw2: track 0.00 -> 60.1 mm
- net sw3: track 0.00 -> 49.2 mm
- net Net-(D13-DIN): track 0.00 -> 43.4 mm, vias 0 -> 2
- net sw1: track 0.00 -> 35.6 mm
- net sw4: track 0.00 -> 27.7 mm
- net Din: track 0.00 -> 9.36 mm
Other:
- board size 127 x 94.5 mm -> 37.4 x 40.6 mm

Commit message: work
Parts:
- added G***: LOGO, LOGO, F.Cu at (-89.8, 130.7)
- added G***: LOGO, LOGO, B.Cu at (-89.8, 130.7)
- added J2: Conn_01x01_Socket, Connector_PinHeader_2.54mm:PinHeader_1x01_P2.54mm_Vertical, F.Cu at (-64.3, 119.2)
- J7: footprint Connector_PinHeader_2.54mm:PinHeader_1x07_P2.54mm_Vertical -> customs:PinHeader_1x07_P2.54mm_Vertical
Routing:
- net Net-(D16-DOUT): track 0.00 -> 12.2 mm
- added copper zone on F.Cu, net (none)
Other:
- outline, holes or cut-outs redrawn
- board text added: "1"
- board text added: "2"
- board text added: "3"
- board text added: "3v3"
- board text added: "4"
- board text added: "ARGOS CONTROLLER REV 1.0"
- board text added: "ARGOS SWITCH REV 1.0"
- board text added: "DESIGN BY Q. LEBASTARD BASTARDKB 2024"
- board text added: "RGB"
- board text added: "github.com/bastardkb"

Commit message: work
Routing:
- net Net-(D15-DOUT): track 73.1 -> 72.3 mm
- added copper zone on B.Cu, net (none)
Changed lines of the file:
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@@
+	)
+	(segment
+		(start -64.85 130.675)
+		(end -64.85 120.7)
+		(width 0.1)
+		(layer "B.Cu")
+		(net 7)
+	)
+	(segment
+		(start -71.275 101.725)
+		(end -68.7 101.725)
+		(width 0.1)
+		(layer "B.Cu")
+		(net 7)
+	)
+	(segment
+		(start -71.145436 132.25)
+		(end -66.425 132.25)
+		(width 0.1)
+		(layer "B.Cu")
+		(net 7)
+	)
+	(segment
+		(start -68.7 101.725)
+		(end -65.175 105.25)
+		(width 0.1)
+		(layer "B.Cu")
+		(net 7)
+	)
+	(segment
+		(start -77.4 103.332842)
+		(end -76.517158 102.45)
+		(width 0.1)
+		(layer "B.Cu")
+		(net 7)
+	)
+	(segment
+		(start -76.517158 102.45)
+		(end -75.783579 102.45)
+		(width 0.1)
+		(layer "B.Cu")
+		(net 7)
+	)
+	(segment
+		(start -78.05 117.05)
+		(end -78.05 111.682842)
+		(width 0.1)
+		(layer "B.Cu")
+		(net 7)
+	)
+	(segment
+		(start -66.625 117.875)
+		(end -77.225 117.875)
+		(width 0.1)
+		(layer "B.Cu")
+		(net 7)
+	)
+	(segment
+		(start -65.875 119.675)
+		(end -65.875 118.625)
+		(width 0.1)
+		(layer "B.Cu")
+		(net 7)
+	)
+	(segment
+		(start -75.783579 102.45)
+		(end -75.783579 101.716421)
+		(width 0.1)
+		(layer "B.Cu")
+		(net 7)
+	)
+	(segment
+		(start -65.175 105.25)
+		(end -65.175 110.95)
+		(width 0.1)
+		(layer "B.Cu")
+		(net 7)
+	)
+	(segment
+		(start -77.4 111.032842)
+		(end -77.4 103.332842)
+		(width 0.1)
+		(layer "B.Cu")
+		(net 7)
+	)
+	(segment
+		(start -71.766 101.234)
+		(end -71.275 101.725)
+		(width 0.1)
+		(layer "B.Cu")
+		(net 7)
+	)
+	(segment
+		(start -72.045436 129.550544)
+		(end -72.045436 131.35)
+		(width 0.1)
+		(layer "B.Cu")
+		(net 7)
 	)
 	(segment
 		(start -75.301158 101.234)
-		(end -75.783579 101.716421)
-		(width 0.1)
-		(layer "B.Cu")
-		(net 7)
-	)
-	(segment
-		(start -71.766 101.234)
+		(end -71.766 101.234)
+		(width 0.1)
+		(layer "B.Cu")
+		(net 7)
+	)
+	(segment
+		(start -77.225 117.875)
+		(end -78.05 117.05)
+		(width 0.1)
+		(layer "B.Cu")
+		(net 7)
+	)
+	(segment
+		(start -75.783579 101.716421)
 		(end -75.301158 101.234)
 		(width 0.1)
@@
 	)
 	(segment
-		(start -78.05 117.05)
-		(end -77.225 117.875)
-		(width 0.1)
-		(layer "B.Cu")
-		(net 7)
-	)
-	(segment
-		(start -64.85 118.225)
+		(start -78.05 111.682842)
+		(end -77.4 111.032842)
+		(width 0.1)
+		(layer "B.Cu")
+		(net 7)
+	)
+	(segment
+		(start -65.875 118.625)
+		(end -66.625 117.875)
+		(width 0.1)
+		(layer "B.Cu")
+		(net 7)
+	)
+	(segment
+		(start -72.045436 131.35)
+		(end -71.145436 132.25)
+		(width 0.1)
+		(layer "B.Cu")
+		(net 7)
+	)
+	(segment
+		(start -66.425 132.25)
 		(end -64.85 130.675)
 		(width 0.1)
@@
 	)
 	(segment
-		(start -64.85 130.675)
-		(end -66.425 132.25)
-		(width 0.1)
-		(layer "B.Cu")
-		(net 7)
-	)
-	(segment
-		(start -72.045436 131.35)
-		(end -72.045436 129.550544)
-		(width 0.1)
-		(layer "B.Cu")
-		(net 7)
-	)
-	(segment
-		(start -71.275 101.725)
-		(end -71.766 101.234)
-		(width 0.1)
-		(layer "B.Cu")
-		(net 7)
-	)
-	(segment
-		(start -75.783579 102.45)
-		(end -76.517158 102.45)
-		(width 0.1)
-		(layer "B.Cu")
-		(net 7)
-	)
-	(segment
-		(start -66.425 132.25)
-		(end -71.145436 132.25)
-		(width 0.1)
-		(layer "B.Cu")
-		(net 7)
-	)
-	(segment
-		(start -78.05 111.682842)
-		(end -78.05 117.05)
-		(width 0.1)
-		(layer "B.Cu")
-		(net 7)
-	)
-	(segment
-		(start -77.225 117.875)
-		(end -65.2 117.875)
-		(width 0.1)
-		(layer "B.Cu")
-		(net 7)
-	)
-	(segment
-		(start -68.7 101.725)
-		(end -71.275 101.725)
-		(width 0.1)
-		(layer "B.Cu")
-		(net 7)
-	)
-	(segment
-		(start -75.783579 101.716421)
-		(end -75.783579 102.45)
-		(width 0.1)
-		(layer "B.Cu")
-		(net 7)
-	)
-	(segment
-		(start -77.4 111.032842)
-		(end -78.05 111.682842)
-		(width 0.1)
-		(layer "B.Cu")
-		(net 7)
-	)
-	(segment
-		(start -65.175 110.95)
-		(end -65.175 105.25)
-		(width 0.1)
-		(layer "B.Cu")
-		(net 7)
-	)
-	(segment
-		(start -77.4 103.332842)
-		(end -77.4 111.032842)
-		(width 0.1)
-		(layer "B.Cu")
-		(net 7)
-	)
-	(segment
-		(start -71.145436 132.25)
-		(end -72.045436 131.35)
-		(width 0.1)
-		(layer "B.Cu")
-		(net 7)
-	)
-	(segment
-		(start -76.517158 102.45)
-		(end -77.4 103.332842)
-		(width 0.1)
-		(layer "B.Cu")
-		(net 7)
-	)
-	(segment
-		(start -65.2 117.875)
-		(end -64.85 118.225)
-		(width 0.1)
-		(layer "B.Cu")
-		(net 7)
-	)
-	(segment
-		(start -65.175 105.25)
-		(end -68.7 101.725)
+		(start -64.85 120.7)
+		(end -65.875 119.675)
 		(width 0.1)
 		(layer "B.Cu")
@@
 		(net 0)
 		(net_name "")
-		(layer "F.Cu")
+		(layers "F&B.Cu")
 		(name "3V3")
 		(hatch edge 0.508)
@@
 			(thermal_gap 0.7)
 			(thermal_bridge_width 0.2)
-			(island_removal_mode 2)
+			(island_removal_mode 1)
 			(island_area_min 0)
 			(hatch_thickness 0.7)

Commit message: angle PCB
Parts:
- moved SW5 2.19 mm to (-94.3, 100.6), turned to 5 degrees
- moved D14 1.79 mm to (-94.0, 105.1), turned to 5 degrees
- moved C3 1.00 mm to (-78.8, 135.7)
- moved G*** 1.00 mm to (-89.8, 131.7) (x2)
- moved J7 1.00 mm to (-97.3, 131.7)
- moved R3 1.00 mm to (-76.6, 135.7)
- moved SW6 0.54 mm to (-92.7, 119.4), turned to 5 degrees
- moved D13 0.15 mm to (-92.3, 124.0), turned to 5 degrees
Routing:
- net Gnd: track 189.1 -> 191.9 mm
- net Vcc: track 149.4 -> 151.5 mm
- net sw2: track 60.1 -> 61.9 mm
- net sw1: track 35.6 -> 37.5 mm
- net Net-(D13-DIN): track 43.4 -> 45.2 mm
- net sw4: track 27.7 -> 28.7 mm
- net sw3: track 49.2 -> 50.2 mm
- net Net-(D14-DOUT): track 128.4 -> 129.0 mm
Other:
- board size 37.4 x 40.6 mm -> 40.1 x 42.3 mm
- board text removed: "ARGOS CONTROLLER REV 1.0"
- board text removed: "DESIGN BY Q. LEBASTARD BASTARDKB 2024"

Commit message: work
Other:
- outline, holes or cut-outs redrawn
- board text added: "CERN OHL-S v2"
